File: hardware/hardware.kicad_sch (KiCad schematic)
At the start: 18 parts, among them J1 5V, J2 GND, J4 MISO, J5 MOSI, J6 SCK, J7 CS, J8 VIN, J9 VOUT, U1 MAX7456EUI+, Y1 27MHZ

Commit message: fix lines
Parts:
- J4: value MISO -> DIN
- J5: value MOSI -> DOUT
Connections:
- net MISO renamed DIN
- net MOSI renamed DOUT
Changed lines of the file:
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@@
     (stroke (width 0) (type default))
   )
-  (global_label "MISO" (shape input) (at 165.1 31.75 180) (fields_autoplaced)
-    (effects (font (size 1.27 1.27)) (justify right))
-    (property "Intersheetrefs" "${INTERSHEET_REFS}" (at 158.0907 31.6706 0)
-      (effects (font (size 1.27 1.27)) (justify right) hide)
-    )
-  )
-  (global_label "MOSI" (shape input) (at 163.83 83.82 0) (fields_autoplaced)
-    (effects (font (size 1.27 1.27)) (justify left))
-    (property "Intersheetrefs" "${INTERSHEET_REFS}" (at 170.8393 83.8994 0)
+  (global_label "DIN" (shape input) (at 165.1 31.75 180) (fields_autoplaced)
+    (effects (font (size 1.27 1.27)) (justify right))
+    (property "Intersheetrefs" "${INTERSHEET_REFS}" (at 158.9095 31.75 0)
+      (effects (font (size 1.27 1.27)) (justify right) hide)
+    )
+  )
+  (global_label "DOUT" (shape input) (at 163.83 83.82 0) (fields_autoplaced)
+    (effects (font (size 1.27 1.27)) (justify left))
+    (property "Intersheetrefs" "${INTERSHEET_REFS}" (at 171.7138 83.82 0)
       (effects (font (size 1.27 1.27)) (justify left) hide)
     )
@@
     )
   )
-  (global_label "MISO" (shape input) (at 128.27 86.36 180) (fields_autoplaced)
-    (effects (font (size 1.27 1.27)) (justify right))
-    (property "Intersheetrefs" "${INTERSHEET_REFS}" (at 121.2607 86.2806 0)
+  (global_label "DIN" (shape input) (at 128.27 86.36 180) (fields_autoplaced)
+    (effects (font (size 1.27 1.27)) (justify right))
+    (property "Intersheetrefs" "${INTERSHEET_REFS}" (at 122.0795 86.36 0)
       (effects (font (size 1.27 1.27)) (justify right) hide)
     )
@@
     )
   )
-  (global_label "MOSI" (shape input) (at 165.1 35.56 180) (fields_autoplaced)
-    (effects (font (size 1.27 1.27)) (justify right))
-    (property "Intersheetrefs" "${INTERSHEET_REFS}" (at 158.0907 35.4806 0)
+  (global_label "DOUT" (shape input) (at 165.1 35.56 180) (fields_autoplaced)
+    (effects (font (size 1.27 1.27)) (justify right))
+    (property "Intersheetrefs" "${INTERSHEET_REFS}" (at 157.2162 35.56 0)
       (effects (font (size 1.27 1.27)) (justify right) hide)
     )
@@
       (effects (font (size 1.27 1.27)) (justify left))
     )
-    (property "Value" "MOSI" (at 173.99 35.56 0)
+    (property "Value" "DOUT" (at 173.99 35.56 0)
       (effects (font (size 1.27 1.27)) (justify left))
     )
@@
       (effects (font (size 1.27 1.27)) (justify left))
     )
-    (property "Value" "MISO" (at 173.99 31.75 0)
-      (effects (font (size 1.27 1.27)) (justify left))
-    )
+    (property "Value" "DIN" (at 173.99 31.75 0)
+      (effects (font (size 1.27 1.27)) (justify left))
+    )
